File: LoraWAN-Stick.kicad_pcb (KiCad board)
At the start: 2 copper layers, 124.2 x 22.9 mm, 31 parts, among them CN1 JST_2PIN-SMT, P1 USB_OTG, SW1 SPST, U1 FGPMMOPA6H, U2 ATmega32U4-AU, U3 RN2903-I/RM095, U4 SPX3819, U5 MCP73831

Commit message: Fixed LiPo charging, added holes on edges, added pads for external crystal, cleaned up silk screen
Parts:
- added 8MHz1: CRYSTAL_2, Crystals:ABM3, F.Cu at (152.7, 93.5)
- added C7: C, Capacitors_SMD:C_0603_HandSoldering, F.Cu at (150.1, 87.4)
- added C8: C, Capacitors_SMD:C_0603_HandSoldering, F.Cu at (150.1, 89.2)
- added REF**: Measurement_Point_Round-SMD-Pad_Big, misc:Mounting-Hole, F.Cu at (196.6, 75.4)
- added REF**: Measurement_Point_Round-SMD-Pad_Big, misc:Mounting-Hole, F.Cu at (196.6, 92.5)
- added REF**: Measurement_Point_Round-SMD-Pad_Big, misc:Mounting-Hole, F.Cu at (78.5, 92.5)
- U5: footprint misc:MCP73831 -> arthurc:SOT23-5
- moved D3 63.7 mm to (191.5, 94.2)
- moved C5 58.1 mm to (81.8, 77.0)
- moved C6 58.1 mm to (92.7, 82.5)
- moved CN1 58.1 mm to (90.9, 77.3)
- moved SW1 58.1 mm to (90.9, 92.1)
- moved U5 58.1 mm to (82.3, 74.4)
- moved ANT1 58.1 mm to (197.6, 83.9)
- moved C1 58.1 mm to (117.6, 83.8)
- moved C2 58.1 mm to (119.9, 85.3)
- moved C3 58.1 mm to (147.1, 84.6)
- moved C4 58.1 mm to (122.4, 85.3)
- moved D1 58.1 mm to (117.6, 79.2)
- moved D2 58.1 mm to (77.5, 73.4)
- moved JP1 58.1 mm to (144.9, 93.8)
- moved JP2 58.1 mm to (154.1, 83.7)
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Routing:
- net GND: track 269.3 -> 304.9 mm, vias 35 -> 44
- net Net-(8MHz1-Pad1): track 0.00 -> 28.0 mm, vias 0 -> 2
- net Net-(8MHz1-Pad2): track 0.00 -> 21.8 mm, vias 0 -> 2
- net Net-(D3-Pad2): track 8.40 -> 2.67 mm
- net Net-(R4-Pad1): track 3.26 -> 6.48 mm
- net Net-(R5-Pad2): track 5.38 -> 2.77 mm
- net (no net): track 5.10 -> 3.84 mm
- net 3v3: track 164.9 -> 164.0 mm
- net VBUS: track 86.9 -> 87.6 mm
Other:
- board size 124.2 x 22.9 mm -> 124.1 x 22.9 mm
- board text added: "D2"
- board text added: "D4"
- board text added: "LoRaWAN Stick - Rev2 GPS - MTK3339 LoRa - RN2903 uC - 32u4 1/10/2017"
- board text added: "R1"
- board text added: "R4"
- board text added: "R5"
- board text added: "R9"
- board text added: "SPX3819"
- board text removed: "LoRaWAN Stick - Rev1 GPS - MTK3339 LoRa - RN2903 uC - 32u4"
