File: LoraWAN-Stick.sch (KiCad schematic (older format))
At the start: 31 parts, among them CN1 JST_2PIN-SMT, P1 USB_OTG, SW1 SPST, U1 FGPMMOPA6H, U2 ATmega32U4-AU, U3 RN2903-I/RM095, U4 SPX3819, U5 MCP73831

Commit message: Fixed LiPo charging, added holes on edges, added pads for external crystal, cleaned up silk screen
Parts:
- added 8MHz1: CRYSTAL_2, Crystals:ABM3, symbol CRYSTAL_2
- added C7, C8: C, Capacitors_SMD:C_0603_HandSoldering, symbol C
Connections:
- net GND: now also C7.2, C8.2
- net at U2.16 (XTAL2): now also 8MHz1.2, C8.1
- net at U2.17 (XTAL1): now also 8MHz1.1, C7.1
Other:
- note added: "1"
- note added: "Dec 28th, 2016"
- note added: "LoraWAN Stick"
Changed lines of the file:
@@
 Wire Wire Line
 	1050 6800 1050 7100
+Text Notes 7500 7500 0    60   ~ 0
+LoraWAN Stick
+Text Notes 10650 7650 0    60   ~ 0
+1
+Text Notes 8200 7650 0    60   ~ 0
+Dec 28th, 2016
+$Comp
+L CRYSTAL_2 8MHz1
+U 1 1 58763D4A
+P 2150 3300
+F 0 "8MHz1" H 2150 3450 60  0000 C CNN
+F 1 "CRYSTAL_2" H 2150 3150 60  0000 C CNN
+F 2 "Crystals:ABM3" H 2150 3300 60  0001 C CNN
+F 3 "" H 2150 3300 60  0000 C CNN
+	1    2150 3300
+	0    1    1    0
+$EndComp
+Wire Wire Line
+	2800 3100 2800 3200
+Wire Wire Line
+	2150 3500 2800 3500
+Wire Wire Line
+	2800 3500 2800 3300
+$Comp
+L GND #PWR023
+U 1 1 58763F9B
+P 1650 3500
+F 0 "#PWR023" H 1650 3500 30  0001 C CNN
+F 1 "GND" H 1650 3430 30  0001 C CNN
+F 2 "" H 1650 3500 60  0000 C CNN
+F 3 "" H 1650 3500 60  0000 C CNN
+	1    1650 3500
+	1    0    0    -1
+$EndComp
+Connection ~ 2150 3100
+$Comp
+L C C7
+U 1 1 587642B5
+P 2000 3100
+F 0 "C7" H 2025 3200 50  0000 L CNN
+F 1 "C" H 2025 3000 50  0000 L CNN
+F 2 "Capacitors_SMD:C_0603_HandSoldering" H 2038 2950 50  0001 C CNN
+F 3 "" H 2000 3100 50  0000 C CNN
+	1    2000 3100
+	0    1    1    0
+$EndComp
+$Comp
+L C C8
+U 1 1 58764348
+P 2000 3500
+F 0 "C8" H 2025 3600 50  0000 L CNN
+F 1 "C" H 2025 3400 50  0000 L CNN
+F 2 "Capacitors_SMD:C_0603_HandSoldering" H 2038 3350 50  0001 C CNN
+F 3 "" H 2000 3500 50  0000 C CNN
+	1    2000 3500
+	0    1    1    0
+$EndComp
+Wire Wire Line
+	1850 3100 1650 3100
+Wire Wire Line
+	1650 3100 1650 3500
+Wire Wire Line
+	1850 3500 1850 3400
+Wire Wire Line
+	1850 3400 1650 3400
+Connection ~ 1650 3400
+Wire Wire Line
+	2800 3100 2150 3100
 $EndSCHEMATC
